Commit message: Add cheat locomotion, noisy odometry and keyboard/PS5 teleop
- quadruped_gz_plugins: PlanarBodyDriver gz system (force/torque
  velocity tracking from /cmd_vel, leaves z/roll/pitch to physics)
- Ground-truth OdometryPublisher and noisy_odom_node (/odom + TF)
- Fake diagonal leg gait in posture_node, slippery feet in cheat mode
- PS5 teleop via joy + teleop_twist_joy + joy_actions_node
- Enable pytest for quadruped_control so the linters actually run

Co-Authored-By: Claude Opus 5.5 <noreply@anthropic.com>

File: src/go2_description/urdf/go2.gazebo.xacro (robot description, xacro)
@@ -1,16 +1,45 @@
 <?xml version="1.0"?>
-<!-- Gazebo-only extensions: ros2_control plugin and contact properties. -->
+<!-- Gazebo-only extensions: ros2_control plugin, contact properties,
+     ground-truth odometry and (cheat:=true) the planar body driver. -->
 <robot xmlns:xacro="http://www.ros.org/wiki/xacro">
-  <xacro:macro name="go2_gazebo" params="controllers_file">
+  <xacro:macro name="go2_gazebo" params="controllers_file cheat">
     <gazebo>
       <plugin filename="gz_ros2_control-system" name="gz_ros2_control::GazeboSimROS2ControlPlugin">
         <parameters>${controllers_file}</parameters>
       </plugin>
+      <!-- Perfect odometry straight from the simulator, for comparison only. -->
+      <plugin filename="gz-sim-odometry-publisher-system"
+              name="gz::sim::systems::OdometryPublisher">
+        <odom_frame>odom</odom_frame>
+        <robot_base_frame>base_link</robot_base_frame>
+        <odom_topic>/model/go2/ground_truth/odom</odom_topic>
+        <tf_topic>/model/go2/ground_truth/tf</tf_topic>
+        <odom_publish_frequency>50</odom_publish_frequency>
+        <dimensions>3</dimensions>
+      </plugin>
     </gazebo>
-    <!-- Feet: rubber-like friction, stiff but damped contact so the robot doesn't bounce. -->
+    <xacro:if value="${cheat}">
+      <!-- Cheat locomotion: an invisible horizontal push tracking /cmd_vel.
+           See quadruped_gz_plugins/src/planar_body_driver.cpp. -->
+      <gazebo>
+        <plugin filename="PlanarBodyDriver" name="quadruped_gz_plugins::PlanarBodyDriver">
+          <topic>/cmd_vel</topic>
+          <!-- Proportional gains: force = gain * velocity error. Higher = less lag and
+               less steady-state error against foot friction, but a harder push. -->
+          <linear_gain>800</linear_gain>      <!-- N per m/s -->
+          <angular_gain>80</angular_gain>     <!-- N*m per rad/s -->
+          <max_force>150</max_force>          <!-- N -->
+          <max_torque>30</max_torque>         <!-- N*m -->
+          <cmd_timeout>0.5</cmd_timeout>      <!-- s: stop if /cmd_vel goes quiet -->
+        </plugin>
+      </gazebo>
+    </xacro:if>
+    <!-- Feet: rubber-like friction, stiff but damped contact so the robot doesn't bounce.
+         In cheat mode the feet are slippery so they glide instead of dragging. -->
+    <xacro:property name="foot_mu" value="${0.1 if cheat else 1.0}"/>
     <xacro:macro name="go2_foot_contact" params="leg">
       <gazebo reference="${leg}_foot">
-        <mu1>1.0</mu1>
-        <mu2>1.0</mu2>
+        <mu1>${foot_mu}</mu1>
+        <mu2>${foot_mu}</mu2>
         <kp>1.0e6</kp>
         <kd>100.0</kd>

File: src/go2_description/urdf/go2.urdf.xacro (robot description, xacro)
@@ -2,8 +2,10 @@
 <!-- Top-level Unitree Go2 description.
      sim:=true adds the ros2_control interface and the Gazebo plugins;
-     controllers_file is the ros2_control parameters YAML handed to gz_ros2_control. -->
+     controllers_file is the ros2_control parameters YAML handed to gz_ros2_control;
+     cheat:=true moves the body with an invisible push instead of walking. -->
 <robot name="go2" xmlns:xacro="http://www.ros.org/wiki/xacro">
   <xacro:arg name="sim" default="false"/>
   <xacro:arg name="controllers_file" default=""/>
+  <xacro:arg name="cheat" default="true"/>
   <xacro:include filename="$(find go2_description)/urdf/go2_body.xacro"/>
   <xacro:go2_body/>
@@ -12,5 +14,5 @@
     <xacro:include filename="$(find go2_description)/urdf/go2.gazebo.xacro"/>
     <xacro:go2_ros2_control/>
-    <xacro:go2_gazebo controllers_file="$(arg controllers_file)"/>
+    <xacro:go2_gazebo controllers_file="$(arg controllers_file)" cheat="$(arg cheat)"/>
   </xacro:if>
 </robot>
